File: schematics/bramble/pmu.kicad_sch (KiCad schematic)
At the start: 9 parts, among them J1 Conn_ARM_JTAG_SWD_10, SW1 SW_Push, U1 STM32L010F4P6, Y1 SG-3030CM

Commit message: Udpate schematics
Parts:
- removed J1: Conn_ARM_JTAG_SWD_10, symbol Connector:Conn_ARM_JTAG_SWD_10
- added D1: LED_Dual_AKA, symbol Device:LED_Dual_AKA
- added J1: Conn_01x05_Pin, Connector_JST:JST_EH_B5B-EH-A_1x05_P2.50mm_Vertical, symbol Connector:Conn_01x05_Pin
- C1: value C -> 100nF
Connections:
- net GND: now also U1.15 (VSS), D1.2 (K), J1.5 (Pin_5)
- net NRST: now also J1.4 (Pin_4)
- net STM32_SUPPLY: now also J1.1 (Pin_1)
- net at U1.19 (PA13): now also J1.3 (Pin_3)
- net at U1.20 (PA14): now also J1.2 (Pin_2)
- net at U1.10 (PA4): now also D1.1 (A1)
- net at U1.11 (PA5): now also D1.3 (A2)
- net 3.3V_SUPPLY_ON: now reaches U1.7 (PA1)
Other:
- moved on the sheet: U1

Commit message: Shematics: split out valve indexer, copy design from rp2040 feather
Parts:
- removed SW1: SW_Push, symbol Switch:SW_Push
- added SW4: SW_MEC_5E, Button_Switch_SMD:SW_SPST_EVQP2_MiddlePushTravel_H2.5mm, symbol Switch:SW_MEC_5E
- C3: renamed from C2; footprint (none) -> Capacitor_SMD:C_0805_2012Metric
- C4: renamed from C3; footprint (none) -> Capacitor_SMD:C_0805_2012Metric
- C5: renamed from C4; footprint (none) -> Capacitor_SMD:C_0805_2012Metric
- C6: renamed from C1; footprint (none) -> Capacitor_SMD:C_0805_2012Metric
- D1: footprint (none) -> LED_THT:LED_D3.0mm-3
- R11: renamed from R21; footprint (none) -> Resistor_SMD:R_0805_2012Metric
- U3: renamed from U1; footprint TSSOP20 -> Package_SO:TSSOP-20_4.4x6.5mm_P0.65mm
Connections:
- net GND: now also SW4.3 (K), SW4.4 (A)
- net NRST: now also SW4.1, SW4.2
Other:
- moved on the sheet: D1
