File: schematics/bramble/valve_indexer.kicad_sch (KiCad schematic)
At the start: 34 parts, among them M1 Motor_DC, M2 Motor_DC, M3 Motor_DC, M4 Motor_DC, Q1 IRLB3813PBF, Q10 IRLB8721PBF, Q2 IRLB3813PBF, Q3 IRF9540N, Q4 IRF9540N, Q5 IRLB3813PBF, Q6 IRLB3813PBF, Q7 IRLB8721PBF, Q8 IRLB8721PBF, Q9 IRLB8721PBF

Commit message: Update valve controller pin mapping for Feather RP2040
- Changed H-bridge pins to use analog-capable GPIOs:
  - MOTOR_LO_1: GPIO26 (A0)
  - MOTOR_LO_2: GPIO27 (A1)
  - MOTOR_HI_1: GPIO28 (A2)
  - MOTOR_HI_2: GPIO29 (A3)
- Updated valve count from 4 to 2 valves
- Valve control pins now on GPIO24 and GPIO25
- This avoids conflict with default I2C pins (GPIO2/3)

🤖 Generated with [Claude Code](https://claude.ai/code)

Co-Authored-By: Claude <noreply@anthropic.com>
Connections:
- no-connect marks 0 -> 6
Changed lines of the file:
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@@
 		(color 0 0 0 0)
+	)
+	(no_connect
+		(at 236.22 116.84)
+	)
+	(no_connect
+		(at 222.25 3.81)
+	)
+	(no_connect
+		(at 179.07 -38.1)
+	)
+	(no_connect
+		(at 243.84 95.25)
+	)
+	(no_connect
+		(at 119.38 8.89)
+	)
+	(no_connect
+		(at 273.05 140.97)
 	)
 	(wire
