File: schematics/bramble/valve_indexer.kicad_sch (KiCad schematic)
At the start: 34 parts, among them M1 Motor_DC, M2 Motor_DC, M3 Motor_DC, M4 Motor_DC, Q1 IRLB3813PBF, Q10 IRLB8721PBF, Q2 IRLB3813PBF, Q3 IRF9540N, Q4 IRF9540N, Q5 IRLB3813PBF, Q6 IRLB3813PBF, Q7 IRLB8721PBF, Q8 IRLB8721PBF, Q9 IRLB8721PBF

Commit message: Udpate schematics
Parts:
- removed Q10, Q7, Q8, Q9: IRLB8721PBF, Package_TO_SOT_THT:TO-220-3_Vertical, symbol Transistor_FET:IRLB8721PBF
- removed R15, R16: 100, symbol Device:R_US
- removed R17, R20: 10k, symbol Device:R_US
- added U4, U5, U6, U7: TLP222A, Package_DIP:DIP-4_W7.62mm, symbol Relay_SolidState:TLP222A
- R13, R14: value 100 -> 170
- R18, R19: value 10k -> 170
Connections:
- net GND: now also U4.2, U5.2, U6.2, U7.2; no longer R18.2, R19.2
- net M+: now also Q3.2 (D)
- net M-: now also U4.3, U5.3, U6.3, U7.3
- net VALVE_1: now also R18.1; no longer R13.2
- net VALVE_2: now also R19.1; no longer R14.2
- net VALVE_3: now also R13.1
- net VALVE_4: now also R14.1
- net at M1.2 (-): now also U4.4
- net at M4.2 (-): now also U7.4
- net at M2.2 (-): now also U5.4
- net at M3.2 (-): now also U6.4
- new net: R18.2, U4.1
- new net: R19.2, U5.1
- new net: R13.2, U6.1
- new net: R14.2, U7.1
- no-connect marks 6 -> 5
Other:
- moved on the sheet: M1, M2, M3, M4, Q3
