File: schematics/bramble/bramble.kicad_sch (KiCad schematic)
At the start: 10 parts, among them U2 TDN_5-0910WISM, U3 Opamp_Quad

Commit message: Udpate schematics
Parts:
- added Q7: IRLB3813PBF, Package_TO_SOT_THT:TO-220-3_Vertical, symbol Transistor_FET:IRLB8721PBF
- added R15: 100, symbol Device:R_US
- added R16: 10k, symbol Device:R_US
Connections:
- net +9V: now also Q7.3 (S); no longer U2.1 (+VIN)
- net GND: now also U2.2 (-VIN), R16.2
- new net: Q7.2 (D), U2.1 (+VIN)
- new net: Q7.1 (G), R15.1, R16.1
- new net 3.3_SUPPLY_ON: R15.2
Other:
- moved on the sheet: U2

Commit message: Shematics: split out valve indexer, copy design from rp2040 feather
Parts:
- removed Q7: IRLB3813PBF, Package_TO_SOT_THT:TO-220-3_Vertical, symbol Transistor_FET:IRLB8721PBF
- added C1, C2: 10uF, Capacitor_SMD:C_0805_2012Metric, symbol Adafruit Feather RP2040 RFM-eagle-import:CAP_CERAMIC0805-NOOUTLINE
- added Q1: DMN3300U, Package_TO_SOT_SMD:SOT-23, symbol Transistor_FET:DMN3300U
- R1: renamed from R15; footprint (none) -> Resistor_SMD:R_0805_2012Metric
- R10: renamed from R29; footprint (none) -> Resistor_SMD:R_0805_2012Metric
- R2: renamed from R16; footprint (none) -> Resistor_SMD:R_0805_2012Metric
- R3: renamed from R26; footprint (none) -> Resistor_SMD:R_0805_2012Metric
- R4: renamed from R25; footprint (none) -> Resistor_SMD:R_0805_2012Metric
- R5: renamed from R24; footprint (none) -> Resistor_SMD:R_0805_2012Metric
- R6: renamed from R22; footprint (none) -> Resistor_SMD:R_0805_2012Metric
- R7: renamed from R23; footprint (none) -> Resistor_SMD:R_0805_2012Metric
- R8: renamed from R27; footprint (none) -> Resistor_SMD:R_0805_2012Metric
- R9: renamed from R28; footprint (none) -> Resistor_SMD:R_0805_2012Metric
- U2: renamed from U3; footprint (none) -> Package_SO:TSSOP-14_4.4x5mm_P0.65mm
- renumbered U2 to U1
Connections:
- net +3.3V: now also C1.1, C2.1
- net +9V: now also Q1.2 (S)
- net GND: now also C1.2, C2.2
- net at U1.1 (+VIN): now also Q1.3 (D)
- net at R1.1, R2.1: now also Q1.1 (G)
Other:
- removed sheet valve_indexer
- added sheet rp2040 (rp2040.kicad_sch)
