File: schematics/bramble/bramble_valve_indexer/bramble_valve_indexer.kicad_sch (KiCad schematic)
At the start: 31 parts

Commit message: Shematics: split out valve indexer, copy design from rp2040 feather
Parts:
- removed M?: 1729128, footprints:CONN_1729128_PXC, symbol 2025-11-01_13-33-45:1729128
- removed U? (x4): TLP222A, Package_DIP:DIP-4_W7.62mm, symbol Relay_SolidState:TLP222A
- added H1, H2, H3, H4: MountingHole, MountingHole:MountingHole_3mm_Pad, symbol Mechanical:MountingHole
- added J1: Conn_02x05_Odd_Even, Connector_PinHeader_2.54mm:PinHeader_2x05_P2.54mm_Vertical, symbol Connector_Generic:Conn_02x05_Odd_Even
- added K1, K2, K3, K4: VOR1142B4, Package_SO:SSO-4_6.7x5.1mm_P2.54mm_Clearance8mm, symbol 2025-11-05_14-05-54:VOR1142B4
- Q2, Q4, Q8: renamed from Q?; value AO3400 -> DMN3300U
- R17: renamed from R?; footprint (none) -> Capacitor_SMD:C_0805_2012Metric
- gave numbers to parts that had none: 22
Connections:
- net +9V: now also J1.1 (Pin_1)
- net GND: now also J1.10 (Pin_10), K1.2, K2.2, K3.2, K4.2
- net M-: now also K1.3, K2.3, K3.3, K4.3
- net MOTOR_HI_1: now also J1.2 (Pin_2)
- net MOTOR_HI_2: now also J1.4 (Pin_4)
- net MOTOR_LO_1: now also J1.6 (Pin_6)
- net MOTOR_LO_2: now also J1.8 (Pin_8)
- net VALVE_1: now also J1.3 (Pin_3)
- net VALVE_2: now also J1.5 (Pin_5)
- net VALVE_3: now also J1.7 (Pin_7)
- net VALVE_4: now also J1.9 (Pin_9)
- net at R12.2: now also K1.1
- net at M1.2: now also K1.4
- net at R13.2: now also K2.1
- net at R20.2: now also K3.1
- net at M3.2: now also K3.4
- net at M2.2: now also K2.4
- net at M4.2: now also K4.4
- net at R21.2: now also K4.1
- no-connect marks 5 -> 4
Other:
- moved on the sheet: M1, M2, M3, M4, Q2, Q4, Q6, Q7, Q8, Q9, R14, R15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
