File: schematics/bramble-fan-control/driver.kicad_sch (KiCad schematic)
At the start: 18 parts, among them J2 FAN_1, J3 FAN_2, Q1 BTA16-600SW3G, Q2 BTA16-600SW3G, U1 MOC3021, U2 MOC3021, U3 H11AA1, U4 H11AA1

Commit message: v3 of schematic
Parts:
- Q1: footprint TerminalBlock_Phoenix:TerminalBlock_Phoenix_MKDS-1,5-2-5.08_1x02_P5.08mm_Horizontal -> Package_TO_SOT_THT:TO-220-3_Vertical
Changed lines of the file:
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@@
 			)
 		)
-		(property "Footprint" "TerminalBlock_Phoenix:TerminalBlock_Phoenix_MKDS-1,5-2-5.08_1x02_P5.08mm_Horizontal"
+		(property "Footprint" "Package_TO_SOT_THT:TO-220-3_Vertical"
 			(at 137.16 52.07 0)
 			(effects
