File: schematics/bramble-fan-control/triac_driver.kicad_pcb (KiCad board)
At the start: 2 copper layers, 42 parts, among them J1 Conn_01x03_Pin, J2 FAN_1, J3 FAN_2, J4 Conn_01x04_Pin, J5 Conn_01x05_Pin, Q1 BTA16-600SW3G, Q2 BTA16-600SW3G, SW1 SW_Rotary_1x3_MP, SW2 STM_RESET, U1 MOC3021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

Commit message: v3 of schematic
Parts:
- added H1: MountingHole_Pad, MountingHole:MountingHole_2.5mm_Pad, F.Cu at (16.4, 16.4)
- added H2: MountingHole_Pad, MountingHole:MountingHole_2.5mm_Pad, F.Cu at (70.7, 15.9)
- added H3: MountingHole_Pad, MountingHole:MountingHole_2.5mm_Pad, F.Cu at (16.4, 29.4)
- added H4: MountingHole_Pad, MountingHole:MountingHole_2.5mm_Pad, F.Cu at (16.4, 36.0)
- C8: moved to B.Cu
- Q1: footprint TerminalBlock_Phoenix:TerminalBlock_Phoenix_MKDS-1,5-2-5.08_1x02_P5.08mm_Horizontal -> Package_TO_SOT_THT:TO-220-3_Vertical
- moved PS1 66.0 mm to (108.7, 35.9), turned to 90 degrees
- moved SW1 52.3 mm to (19.2, 77.3)
- moved J2 45.6 mm to (23.6, 105.8)
- moved U4 45.6 mm to (54.8, 49.6)
- moved RV1 45.5 mm to (101.0, 54.9)
- moved C3 39.1 mm to (105.5, 71.2), turned to 90 degrees
- moved J1 32.3 mm to (29.8, 20.1)
- moved R1 32.2 mm to (21.3, 53.2)
- moved U5 31.7 mm to (112.4, 66.3), turned to 180 degrees
- moved J5 30.0 mm to (70.5, 30.6)
- moved J3 29.6 mm to (40.8, 105.8)
- moved R2 28.4 mm to (24.8, 65.5)
- moved C8 27.0 mm to (88.6, 67.8), turned to 180 degrees
- moved U3 24.5 mm to (50.6, 66.0)
- moved Q2 23.1 mm to (40.9, 95.7)
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