File: schematics/bramble-fan-control/triac_driver.kicad_sch (KiCad schematic)
At the start: 5 parts, among them J1 Conn_01x03_Pin, SW1 SW_Rotary_1x3_MP

Commit message: v3 of schematic
Parts:
- added H1, H2, H3, H4: MountingHole_Pad, MountingHole:MountingHole_2.5mm_Pad, symbol Mechanical:MountingHole_Pad
