File: schematics/bramble/bramble-main/bramble.kicad_pcb (KiCad board)
At the start: 2 copper layers, 72.1 x 72.4 mm, 93 parts, among them J1 Conn_01x05_Pin, J2 UART, J3 RPI SWD, J4 U.FL, J5 USB_C_Receptacle_USB2.0_16P, J6 GPIO1, J7 GPIO2, J8 GPIO3, SW1 STM_WAKE, SW2 STM_RESET, SW3 BOOT, SW4 RESET, U1 Opamp_Quad, U2 STM32L031F6P6TR, U3 MCP1700x-120xxMB, U4 FM24CL16B-GTR, U5 RFM95W-915S2, U6 RP2350_80QFN, U7 W25Q16JVSS, U8 MT25QL01GBBB8ESF-0SIT, Y1 Crystal, Y2 ABM8-272-T3

Commit message: Assign JLCPCB parts and regenerate manufacturing files
Updated LCSC part assignments for assembly, regenerated Gerbers,
BOM, and CPL files for JLCPCB fabrication order.

Co-Authored-By: Claude Opus 4.6 <noreply@anthropic.com>
Parts:
- C13, C16, C17, C18, C19, C20, C21, C22, C23, C24, C27: value 100n -> 100nF
- C14, C15: value 4.7u -> 4.7uF
- L1: value 3.3 -> 3.3H; footprint Inductor_SMD:L_0805_2012Metric -> Inductor_SMD:L_Murata_DFE201610P
- MAIN SUPPLY: renamed from MAIN_SUPPLY1
- PMU SUPPLY: renamed from PMU_SUPPLY1
- STM UART: renamed from J3
- moved L1 0.13 mm to (56.1, 38.0)
- renumbered TP4 to +V, SW3 to BOOT, PMU_STATUS1 to PMU, SW4 to RESET, TP3 to RX, TP2 to TX, SW1 to WAKE
Routing:
- net /rp2350B (page 4)/GPIO41_ADC1: track 30.9 -> 34.8 mm, vias 0 -> 2
Other:
- board size 72.1 x 72.4 mm -> 72.1 x 70.7 mm
- board text added: "+3V3"
- board text added: "3V"
- board text added: "GPIO1"
- board text added: "GPIO2"
- board text added: "GPIO3"
- board text added: "P1"
- board text added: "P2"
- board text added: "RESET"
- board text added: "RPI"
- board text added: "S"
- board text added: "TAP"
- board text removed: "GPIO"
- board text removed: "RPI STATUS"
