File: schematics/bramble/bramble-main/bramble.kicad_pcb (KiCad board)
At the start: 2 copper layers, 72.1 x 70.7 mm, 93 parts, among them J1 Conn_01x05_Pin, J2 UART, J4 U.FL, J5 USB_C_Receptacle_USB2.0_16P, J6 GPIO1, J7 GPIO2, J8 GPIO3, SW2 STM_RESET, U1 Opamp_Quad, U2 STM32L031F6P6TR, U3 MCP1700x-120xxMB, U4 FM24CL16B-GTR, U5 RFM95W-915S2, U6 RP2350_80QFN, U7 W25Q16JVSS, U8 MT25QL01GBBB8ESF-0SIT, Y1 Crystal, Y2 ABM8-272-T3

Commit message: Update connector values and regenerate manufacturing files
Set JST PH power connector values to B2B-PH-K-S, fix reference
designator numbering, and assign remaining JLCPCB parts. Regenerated
Gerbers, BOM, and CPL for fabrication.
Parts:
- J3: renamed from STM UART
- MAIN SUPPLY: value ~ -> B2B-PH-K-S
- PMU SUPPLY: value ~ -> B2B-PH-K-S
- renumbered PMU to PMU_STATUS1, WAKE to SW1, BOOT to SW3, RESET to SW4, TX to TP2, RX to TP3, +V to TP4
Routing:
- net /pmu/3V3_POWER_ON: track 87.1 -> 67.7 mm
- net Net-(JP1-B): track 108.0 -> 105.2 mm
- net (no net): track 1.01 -> 0.00 mm
- net Net-(C26-Pad1): track 3.55 -> 2.80 mm
- net /rp2350B (page 4)/GPIO43_ADC3: track 32.7 -> 32.0 mm
- net +9V: track 174.2 -> 173.7 mm
- net Net-(J1-Pin_2): track 69.6 -> 69.1 mm
