File: schematics/bramble/bramble-main/bramble.kicad_pcb (KiCad board)
At the start: 2 copper layers, 72.1 x 70.7 mm, 93 parts, among them J1 Conn_01x05_Pin, J2 UART, J3 RPI SWD, J4 U.FL, J5 USB_C_Receptacle_USB2.0_16P, J6 GPIO1, J7 GPIO2, J8 GPIO3, SW1 STM_WAKE, SW2 STM_RESET, SW3 BOOT, SW4 RESET, U1 Opamp_Quad, U2 STM32L031F6P6TR, U3 MCP1700x-120xxMB, U4 FM24CL16B-GTR, U5 RFM95W-915S2, U6 RP2350_80QFN, U7 W25Q16JVSS, U8 MT25QL01GBBB8ESF-0SIT, Y1 Crystal, Y2 ABM8-272-T3

Commit message: chore(schematics): update bramble v5 main board
Updates PCB, schematics, gerbers, BOM/CPL, and JLCPCB project for
the bramble-v5 hardware revision.

Co-Authored-By: Claude Opus 4.7 (1M context) <noreply@anthropic.com>
Parts:
- added kibuzzard-69F15CED: G***, kibuzzard-69F15CED, F.Cu at (76.2, 42.4)
- added kibuzzard-69F15D28: G***, kibuzzard-69F15D28, F.Cu at (73.5, 42.4)
- added kibuzzard-69F15D48: G***, kibuzzard-69F15D48, F.Cu at (30.2, 69.0)
- added kibuzzard-69F15D48: G***, kibuzzard-69F15D48, F.Cu at (76.7, 50.8)
- added kibuzzard-69F15D5F: G***, kibuzzard-69F15D5F, F.Cu at (74.0, 50.8)
- added kibuzzard-69F15D5F: G***, kibuzzard-69F15D5F, F.Cu at (25.4, 79.9)
- added kibuzzard-69F15DA2: G***, kibuzzard-69F15DA2, F.Cu at (56.5, 68.5)
- added kibuzzard-69F1F93E: G***, kibuzzard-69F1F93E, F.Cu at (64.8, 72.5)
- added kibuzzard-69F1F948: G***, kibuzzard-69F1F948, F.Cu at (50.6, 72.7)
- added kibuzzard-69F1FA9E: G***, kibuzzard-69F1FA9E, F.Cu at (15.6, 37.8)
- added kibuzzard-69F1FABA: G***, kibuzzard-69F1FABA, F.Cu at (19.4, 16.2)
- added kibuzzard-69F1FACD: G***, kibuzzard-69F1FACD, F.Cu at (56.5, 13.8)
- added kibuzzard-69F1FACD: G***, kibuzzard-69F1FACD, F.Cu at (23.2, 13.3)
- added kibuzzard-69F1FAE9: G***, kibuzzard-69F1FAE9, F.Cu at (33.1, 13.4)
- added kibuzzard-69F1FB08: G***, kibuzzard-69F1FB08, F.Cu at (56.5, 20.8)
- added kibuzzard-69F1FB2A: G***, kibuzzard-69F1FB2A, F.Cu at (56.6, 21.9)
- added kibuzzard-69F1FB2A: G***, kibuzzard-69F1FB2A, F.Cu at (15.8, 39.0)
- added kibuzzard-69F1FB3C: G***, kibuzzard-69F1FB3C, F.Cu at (64.3, 16.9)
- added kibuzzard-69F1FB43: G***, kibuzzard-69F1FB43, F.Cu at (69.7, 16.8)
- added kibuzzard-69F1FB5C: G***, kibuzzard-69F1FB5C, F.Cu at (61.0, 34.3)
- added kibuzzard-69F1FB6D: G***, kibuzzard-69F1FB6D, F.Cu at (61.0, 26.7)
- added kibuzzard-69F1FBEC: G***, kibuzzard-69F1FBEC, B.Cu at (38.1, 35.6)
- added kibuzzard-69F1FC5E: G***, kibuzzard-69F1FC5E, B.Cu at (34.9, 35.6)
- added kibuzzard-69F204CF: G***, kibuzzard-69F204CF, F.Cu at (20.0, 28.9)
- added kibuzzard-69F204DC: G***, kibuzzard-69F204DC, F.Cu at (20.0, 24.9)
- added kibuzzard-69F209F9: G***, kibuzzard-69F209F9, F.Cu at (57.9, 48.2)
- added kibuzzard-69F20A0D: G***, kibuzzard-69F20A0D, F.Cu at (69.7, 48.0)
- added kibuzzard-69F20A1A: G***, kibuzzard-69F20A1A, F.Cu at (69.0, 22.2)
- L1: value 3.3H -> 3.3uH
- MAIN_SUPPLY1: renamed from MAIN SUPPLY; value B2B-PH-K-S -> B2B-PH-K-S
- PMU_SUPPLY1: renamed from PMU SUPPLY; value B2B-PH-K-S -> B2B-PH-K-S
- R23: value 10K -> 10k
- U5: value RFM95W-915S2 -> NiceRF Lora1262
- renumbered SW2 to STM_RESET1, SW1 to STM_WAKE1, SW3 to SW1, SW4 to SW2
Connections:
- J5 pad B6: unconnected-(J5-D+-PadB6) -> /rp2350B (page 4)/D+
- J5 pad B7: unconnected-(J5-D--PadB7) -> /rp2350B (page 4)/D-
- U2 pad 10: Net-(PMU_STATUS1-DIN) -> unconnected-(U2-PA4-Pad10)
- U2 pad 11: unconnected-(U2-PA5-Pad11) -> Net-(PMU_STATUS1-DIN)
- U5 pad 11: /rp2350B (page 4)/RFM_IO2 -> unconnected-(U5-DIO3-Pad11)
- U5 pad 12: /rp2350B (page 4)/RFM_IO1 -> unconnected-(U5-Pad12)
- U5 pad 14: /rp2350B (page 4)/RFM_IO5 -> unconnected-(U5-Pad14)
- U5 pad 15: /rp2350B (page 4)/RFM_IO4 -> /rp2350B (page 4)/RFM_IO1
- U5 pad 16: /rp2350B (page 4)/RFM_IO3 -> /rp2350B (page 4)/RFM_BUSY
- U5 pad 7: /rp2350B (page 4)/RFM_IO0 -> unconnected-(U5-Pad7)
- U6 pad 13: /rp2350B (page 4)/MOSI -> /rp2350B (page 4)/SCK
- U6 pad 14: /rp2350B (page 4)/SCK -> /rp2350B (page 4)/MOSI
- U6 pad 17: /rp2350B (page 4)/RFM_IO0 -> unconnected-(U6-GPIO17-Pad17)
- U6 pad 18: /rp2350B (page 4)/RFM_IO2 -> /rp2350B (page 4)/RFM_BUSY
Routing:
- net /rp2350B (page 4)/RFM_IO2: track 34.9 -> 0.00 mm
- net /rp2350B (page 4)/RFM_IO0: track 30.4 -> 0.00 mm
- net /rp2350B (page 4)/RFM_BUSY: track 0.00 -> 29.4 mm
- net Net-(PMU_STATUS1-DIN): track 36.7 -> 53.8 mm
- net /rp2350B (page 4)/RFM_IO1: track 33.1 -> 21.3 mm
- net /rp2350B (page 4)/MOSI: track 23.9 -> 32.4 mm
- net +3V3: track 424.4 -> 430.3 mm
- net /rp2350B (page 4)/D+: track 14.7 -> 18.8 mm
- net /rp2350B (page 4)/D-: track 14.7 -> 16.6 mm
- net VBUS: track 84.5 -> 85.6 mm
- net unconnected-(U2-PA4-Pad10): track 0.00 -> 0.74 mm
Other:
- board text added: "v0.5, April 2026 E. E. Beerepoot"
- board text removed: "+3V3"
- board text removed: "3V"
- board text removed: "GPIO1"
- board text removed: "GPIO2"
- board text removed: "GPIO3"
- board text removed: "RESET"
- board text removed: "RPI"
- board text removed: "RPI SWD"
- board text removed: "STM DEBUG"
- board text removed: "TAP"
- board text removed: "v0.4, March 2026 E. E. Beerepoot"
