File: schematics/bramble/bramble-main/rp2040.kicad_sch (KiCad schematic)
At the start: 41 parts, among them IC1 RP2040_QFN56, J3 Conn_01x03, J4 USB_C_Receptacle_USB2.0_16P, J5 U.FL, J6 Conn_02x06_Odd_Even, SW2 BOOT, SW3 RESET, U4 RFM95W-915S2, U5 W25Q16JVSS, U6 MT25QL01GBBB8ESF-0SIT, Y2 Crystal

Commit message: Checking in v4 schematic/board prior to attempting jlcpcb run
Parts:
- removed C10, C11: 8pF, Capacitor_SMD:C_0805_2012Metric, symbol Adafruit Feather RP2040 RFM-eagle-import:CAP_CERAMIC_0402NO
- removed C12, C15, C16, C18, C22: 1uF, Capacitor_SMD:C_0805_2012Metric, symbol Adafruit Feather RP2040 RFM-eagle-import:CAP_CERAMIC_0402NO
- removed C13, C14, C17, C19, C20, C21, C9: 0.1uF, Capacitor_SMD:C_0805_2012Metric, symbol Adafruit Feather RP2040 RFM-eagle-import:CAP_CERAMIC_0402NO
- removed IC1: RP2040_QFN56, RP2040:RP2040-QFN-56, symbol Adafruit Feather RP2040 RFM-eagle-import:RP2040_QFN56
- removed R16, R19, R20, R25: 10K, Resistor_SMD:R_0805_2012Metric, symbol Adafruit Feather RP2040 RFM-eagle-import:RESISTOR_0402NO
- removed R18: 1K, Resistor_SMD:R_0805_2012Metric, symbol Adafruit Feather RP2040 RFM-eagle-import:RESISTOR_0402NO
- removed R21, R22: 22 ohm, Resistor_SMD:R_0805_2012Metric, symbol Adafruit Feather RP2040 RFM-eagle-import:RESISTOR_0402NO
- removed R23, R24: 5.1K, Resistor_SMD:R_0805_2012Metric, symbol Adafruit Feather RP2040 RFM-eagle-import:RESISTOR_0402NO
- removed U$1, U$2, U$3, U$4: MOUNTINGHOLE2.5, MountingHole:MountingHole_2.5mm_Pad, symbol Adafruit Feather RP2040 RFM-eagle-import:MOUNTINGHOLE2.5
- removed Y2: Crystal, Crystal:Crystal_SMD_Abracon_ABM3-2Pin_5.0x3.2mm_HandSoldering, symbol Device:Crystal
- added C11, C12: 4.7uF, Capacitor_SMD:C_0402_1005Metric, symbol Device:C
- added C13, C16, C17, C18, C19, C20, C21, C22, C23, C24, C27: 100n, Capacitor_SMD:C_0402_1005Metric, symbol Device:C
- added C14, C15: 4.7u, Capacitor_SMD:C_0402_1005Metric, symbol Device:C
- added C25, C26: 15p, Capacitor_SMD:C_0402_1005Metric, symbol Device:C
- added H1, H2, H3, H4: MountingHole, MountingHole:MountingHole_3.5mm_Pad, symbol Mechanical:MountingHole
- added J7: GPIO2, Connector_IDC:IDC-Header_2x06_P2.54mm_Vertical, symbol Connector_Generic:Conn_02x06_Odd_Even
- added J8: GPIO3, Connector_IDC:IDC-Header_2x06_P2.54mm_Vertical, symbol Connector_Generic:Conn_02x06_Odd_Even
- added L1: 3.3, Inductor_SMD:L_0805_2012Metric, symbol Device:L
- added R11, R12: 10k, Capacitor_SMD:C_0402_1005Metric, symbol Device:R_US
- added R13: 33, Capacitor_SMD:C_0402_1005Metric, symbol Device:R_US
- added R14, R15: 100, Capacitor_SMD:C_0402_1005Metric, symbol Device:R_US
- added R16, R21, R22: 1K, Capacitor_SMD:C_0402_1005Metric, symbol Device:R_US
- added R18, R19: 27, Resistor_SMD:R_0603_1608Metric, symbol Device:R_US
- added R20: 5.1K, Capacitor_SMD:C_0402_1005Metric, symbol Device:R_US
- added R23: 10K, Capacitor_SMD:C_0402_1005Metric, symbol Device:R_US
- added U6: RP2350_80QFN, RP2350_80QFN_minimal:RP2350-QFN-80-1EP_10x10_P0.4mm_EP3.4x3.4mm_ThermalVias, symbol MCU_RaspberryPi_RP2350:RP2350_80QFN
- added Y2: ABM8-272-T3, Crystal:Crystal_SMD_3225-4Pin_3.2x2.5mm, symbol Device:Crystal_GND24
- J3: value Conn_01x03 -> RPI SWD; footprint Connector_PinHeader_2.54mm:PinHeader_1x03_P2.54mm_Vertical -> Connector_JST:JST_SH_BM03B-SRSS-TB_1x03-1MP_P1.00mm_Vertical
- J5: renamed from J4; footprint Connector_USB:USB_C_Receptacle_GCT_USB4110 -> Connector_USB:USB_C_Receptacle_G-Switch_GT-USB-7051x
- J6: value Conn_02x06_Odd_Even -> GPIO1; footprint Connector_PinHeader_2.54mm:PinHeader_2x06_P2.54mm_Vertical -> Connector_IDC:IDC-Header_2x06_P2.54mm_Vertical
- R17: value 1k -> 1K; footprint Resistor_SMD:R_0805_2012Metric -> Capacitor_SMD:C_0402_1005Metric
- renumbered D2 to D1, J5 to J4, SW2 to SW3, SW3 to SW4, U4 to U5, U5 to U7, U6 to U8
Connections:
- net SWDIO is gone; now on net GND: J3.2 (Pin_2)
- net +3V3: now also J6.1 (Pin_1), C11.1, C17.1, C18.1, C19.1, C20.1, C21.1, C22.1, C23.1, C24.1, C27.1, J7.1 (Pin_1), J8.1 (Pin_1), R11.2, R12.2, R13.1, R23.1, U6.15 (IOVDD), U6.24 (IOVDD), U6.29 (IOVDD), U6.41 (IOVDD), U6.5 (IOVDD), U6.50 (IOVDD), U6.59 (ADC_AVDD), U6.60 (IOVDD), U6.64 (VREG_VIN), U6.68 (USB_OTP_VDD), U6.69 (QSPI_IOVDD), U6.76 (IOVDD); no longer J6.2 (Pin_2)
- net +9V: now also J6.2 (Pin_2), J7.2 (Pin_2), J8.2 (Pin_2); no longer J6.1 (Pin_1)
- net D+: now also J5.A6 (D+), R18.2
- net D-: now also J5.A7 (D-), R19.2
- net GND: now also R17.1, U5.SH (SHIELD), C11.2, C12.2, C13.2, C14.2, C15.2, C16.2, C17.2, C18.2, C19.2, C20.2, C21.2, C22.2, C23.2, C24.2, C25.2, C26.2, C27.2, J7.12 (Pin_12), J8.12 (Pin_12), R20.2, R21.2, U6.62 (VREG_PGND), U6.81 (GND), Y2.2, Y2.4; no longer J3.3 (Pin_3), SW4.2
- net MISO: now also U6.11 (GPIO12); no longer U8.8 (DQ1)
- net MOSI: now also U6.13 (GPIO14); no longer U8.15 (DQ0)
- net MOTOR_HI_1: now also J6.10 (Pin_10), U6.36 (GPIO28); no longer J6.4 (Pin_4)
- net MOTOR_HI_2: now also J6.8 (Pin_8), U6.38 (GPIO30); no longer J6.6 (Pin_6)
- net MOTOR_LO_1: now also J6.6 (Pin_6), U6.40 (GPIO32); no longer J6.8 (Pin_8)
- net MOTOR_LO_2: now also J6.4 (Pin_4), U6.43 (GPIO34); no longer J6.10 (Pin_10)
- net MT25_CS: now also U6.78 (GPIO1)
- net MT25_RESET: now also U6.2 (GPIO5)
- net QSPI_D0: now also U6.72 (QSPI_SD0)
- net QSPI_D1: now also U6.74 (QSPI_SD1)
- net QSPI_D2: now also U6.73 (QSPI_SD2)
- net QSPI_D3: now also U6.70 (QSPI_SD3)
- net QSPI_SCK: now also U6.71 (QSPI_SCLK)
- net RFM_CS: now also R12.1, U6.8 (GPIO10)
- net RFM_IO0: now also U5.7 (DIO5), U6.17 (GPIO17); no longer U5.14 (DIO0)
- net RFM_IO1: now also U5.12 (DIO4), U6.19 (GPIO19); no longer U5.15 (DIO1)
- net RFM_IO2: now also U5.11 (DIO3), U6.18 (GPIO18); no longer U5.16 (DIO2)
- net RFM_IO3: now also U5.16 (DIO2); no longer U5.11 (DIO3)
- net RFM_IO4: now also U5.15 (DIO1); no longer U5.12 (DIO4)
- net RFM_IO5: now also U5.14 (DIO0); no longer U5.7 (DIO5)
- net RFM_RST: now also R11.1, U6.16 (GPIO16)
- net RGB_LED: now also U6.1 (GPIO4)
- net RX: now also U6.7 (GPIO9)
- net SCK: now also U6.14 (GPIO15); no longer U8.16 (C)
- net TX: now also U6.6 (GPIO8)
- net VALVE_1: now also U6.37 (GPIO29)
- net VALVE_2: now also U6.39 (GPIO31)
- net VALVE_3: now also U6.44 (GPIO35)
- net VALVE_4: now also U6.42 (GPIO33)
- net VBUS: now also U6.3 (GPIO6)
- net VDD: now also J7.11 (Pin_11), J8.11 (Pin_11)
- net at D1.2 (A): now also R16.2
- net at J5.B5 (CC2): now also R20.1
- net at R17.2: now also SW4.2
- net at J5.A5 (CC1): now also R21.1
- net QSPI_CS renamed QSPI_SS
- net QSPI_SS: now also R16.1, R23.2, U6.75 (QSPI_SS)
- net SWCLK: no longer names the net of J3.1 (Pin_1)
- net SWCLK: now also R14.1
- net ~{RESET} renamed RUN
- net RUN: now also U6.35 (RUN)
- new net: C26.1, R22.1, Y2.3
- new net: R14.2, U6.33 (SWCLK)
- new net: R18.1, U6.67 (USB_DP)
- new net: R15.2, U6.34 (SWD)
- new net: R19.1, U6.66 (USB_DM)
- new net: J3.3 (Pin_3), R15.1
- new net +1V1: C12.1, C13.1, C15.1, C16.1, L1.1, U6.10 (DVDD), U6.32 (DVDD), U6.51 (DVDD), U6.65 (VREG_FB)
- new net GPIO20: J8.9 (Pin_9), U6.20 (GPIO20)
- new net GPIO21: J8.10 (Pin_10), U6.21 (GPIO21)
- new net GPIO22: J8.7 (Pin_7), U6.22 (GPIO22)
- new net GPIO23: J8.8 (Pin_8), U6.23 (GPIO23)
- new net GPIO24: J8.5 (Pin_5), U6.25 (GPIO24)
- new net GPIO25: J8.6 (Pin_6), U6.26 (GPIO25)
- new net GPIO26: J8.3 (Pin_3), U6.27 (GPIO26)
- new net GPIO27: J8.4 (Pin_4), U6.28 (GPIO27)
- new net GPIO28: J7.10 (Pin_10), U6.45 (GPIO36)
- new net GPIO29: J7.9 (Pin_9), U6.46 (GPIO37)
- new net GPIO30: J7.8 (Pin_8), U6.47 (GPIO38)
- new net GPIO31: J7.7 (Pin_7), U6.48 (GPIO39)
- new net GPIO40_ADC0: J7.6 (Pin_6), U6.49 (GPIO40_ADC0)
- new net GPIO41_ADC1: J7.5 (Pin_5), U6.52 (GPIO41_ADC1)
- new net GPIO42_ADC2: J7.4 (Pin_4), U6.53 (GPIO42_ADC2)
- new net GPIO43_ADC3: J7.3 (Pin_3), U6.54 (GPIO43_ADC3)
- new net GPIO44_ADC4: U6.55 (GPIO44_ADC4)
- new net GPIO45_ADC5: U6.56 (GPIO45_ADC5)
- new net GPIO46_ADC6: U6.57 (GPIO46_ADC6)
- new net GPIO47_ADC7: U6.58 (GPIO47_ADC7)
- new net MT25_MISO: U6.77 (GPIO0), U8.8 (DQ1)
- new net MT25_MOSI: U6.80 (GPIO3), U8.15 (DQ0)
- new net MT25_SCK: U6.79 (GPIO2), U8.16 (C)
- new net VREG_AVDD: C14.1, R13.2, U6.61 (VREG_AVDD)
- new net VREG_LX: L1.2, U6.63 (VREG_LX)
- new net XIN: C25.1, U6.30 (XIN), Y2.1
- new net XOUT: R22.2, U6.31 (XOUT)
- no-connect marks 0 -> 16
Other:
- note added: "12MHz Crystal"
- note added: "KEEP CLOSE TO MCU PINS"
- note added: "Make sure R7 and R8 are close to RP2350"
- note removed: "RESET"
- note removed: "RP2040 BYPASS CAPS"
- moved on the sheet: J4, J5, J6, U5
