File: schematics/bramble/bramble-main/rp2040.kicad_sch (KiCad schematic)
At the start: 50 parts, among them J3 RPI SWD, J4 U.FL, J5 USB_C_Receptacle_USB2.0_16P, J6 GPIO1, J7 GPIO2, J8 GPIO3, SW3 BOOT, SW4 RESET, U5 RFM95W-915S2, U6 RP2350_80QFN, U7 W25Q16JVSS, U8 MT25QL01GBBB8ESF-0SIT, Y2 ABM8-272-T3

Commit message: Assign JLCPCB parts and regenerate manufacturing files
Updated LCSC part assignments for assembly, regenerated Gerbers,
BOM, and CPL files for JLCPCB fabrication order.

Co-Authored-By: Claude Opus 4.6 <noreply@anthropic.com>
Parts:
- C13, C16, C17, C18, C19, C20, C21, C22, C23, C24, C27: value 100n -> 100nF
- C14, C15: value 4.7u -> 4.7uF
- L1: value 3.3 -> 3.3H; footprint Inductor_SMD:L_0805_2012Metric -> Inductor_SMD:L_Murata_DFE201610P
Changed lines of the file:
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@@
 			)
 		)
-		(property "Value" "100n"
+		(property "Value" "100nF"
 			(at 212.471 98.933 0)
 			(effects
@@
 			)
 		)
-		(property "Value" "100n"
+		(property "Value" "100nF"
 			(at 143.256 98.933 0)
 			(effects
@@
 			)
 		)
-		(property "Value" "4.7u"
+		(property "Value" "4.7uF"
 			(at 71.501 98.933 0)
 			(effects
@@
 			)
 		)
-		(property "Value" "100n"
+		(property "Value" "100nF"
 			(at 223.901 98.933 0)
 			(effects
@@
 		(fields_autoplaced yes)
 		(property "Reference" "C14"
-			(at 69.85 125.73 0)
+			(at 69.85 125.7299 0)
 			(effects
 				(font
@@
 			)
 		)
-		(property "Value" "4.7u"
-			(at 69.85 128.27 0)
+		(property "Value" "4.7uF"
+			(at 69.85 128.2699 0)
 			(effects
 				(font
@@
 			)
 		)
-		(property "Value" "3.3"
+		(property "Value" "3.3H"
 			(at 46.99 140.9699 0)
 			(effects
@@
 			)
 		)
-		(property "Footprint" "Inductor_SMD:L_0805_2012Metric"
+		(property "Footprint" "Inductor_SMD:L_Murata_DFE201610P"
 			(at 45.72 139.7 0)
 			(effects
@@
 			)
 		)
-		(property "Value" "100n"
+		(property "Value" "100nF"
 			(at 235.331 98.933 0)
 			(effects
@@
 			)
 		)
-		(property "Value" "100n"
+		(property "Value" "100nF"
 			(at 178.181 98.933 0)
 			(effects
@@
 			)
 		)
-		(property "Value" "100n"
+		(property "Value" "100nF"
 			(at 155.321 98.933 0)
 			(effects
@@
 			)
 		)
-		(property "Value" "100n"
+		(property "Value" "100nF"
 			(at 81.661 98.933 0)
 			(effects
@@
 			)
 		)
-		(property "Value" "100n"
+		(property "Value" "100nF"
 			(at 58.801 98.933 0)
 			(effects
@@
 			)
 		)
-		(property "Value" "100n"
+		(property "Value" "100nF"
 			(at 189.611 98.933 0)
 			(effects
@@
 			)
 		)
-		(property "Value" "100n"
+		(property "Value" "100nF"
 			(at 201.041 98.933 0)
 			(effects
@@
 			)
 		)
-		(property "Value" "100n"
+		(property "Value" "100nF"
 			(at 166.751 98.933 0)
 			(effects
