File: schematics/bramble/bramble-main/rp2040.kicad_sch (KiCad schematic)
At the start: 50 parts, among them J3 RPI SWD, J4 U.FL, J5 USB_C_Receptacle_USB2.0_16P, J6 GPIO1, J7 GPIO2, J8 GPIO3, SW3 BOOT, SW4 RESET, U5 RFM95W-915S2, U6 RP2350_80QFN, U7 W25Q16JVSS, U8 MT25QL01GBBB8ESF-0SIT, Y2 ABM8-272-T3

Commit message: chore(schematics): update bramble v5 main board
Updates PCB, schematics, gerbers, BOM/CPL, and JLCPCB project for
the bramble-v5 hardware revision.

Co-Authored-By: Claude Opus 4.7 (1M context) <noreply@anthropic.com>
Parts:
- L1: value 3.3H -> 3.3uH
- R23: value 10K -> 10k
- U5: value RFM95W-915S2 -> NiceRF Lora1262
- renumbered SW3 to SW1, SW4 to SW2
Connections:
- net RFM_IO4 is gone; now on net RFM_IO1: U5.15 (DIO1)
- net D+: now also J5.B6 (D+)
- net D-: now also J5.B7 (D-)
- net MOSI: now also U6.14 (GPIO15); no longer U6.13 (GPIO14)
- net RFM_IO1: no longer U5.12 (DIO4)
- net SCK: now also U6.13 (GPIO14); no longer U6.14 (GPIO15)
- net RFM_IO0: no longer names the net of U5.7
- net RFM_IO0: no longer U6.17 (GPIO17)
- net RFM_IO2: no longer names the net of U5.11 (DIO3)
- net RFM_IO2: no longer U6.18 (GPIO18)
- net RFM_IO3 renamed RFM_BUSY
- net RFM_BUSY: now also U6.18 (GPIO18)
- net RFM_IO5: no longer names the net of U5.14
- no-connect marks 16 -> 15
