File: schematics/bramble/bramble-main/pmu.kicad_sch (KiCad schematic)
At the start: 29 parts, among them J1 Conn_01x05_Pin, J2 UART, SW1 STM_WAKE, SW2 STM_RESET, U2 STM32L031F6P6TR, U3 MCP1700x-120xxMB, U4 FM24CL16B-GTR, Y1 Crystal

Commit message: chore(schematics): update bramble v5 main board
Updates PCB, schematics, gerbers, BOM/CPL, and JLCPCB project for
the bramble-v5 hardware revision.

Co-Authored-By: Claude Opus 4.7 (1M context) <noreply@anthropic.com>
Parts:
- U3: value MCP1700x-120xxMB -> MCP1700T-3002E/MB
- renumbered SW2 to STM_RESET1, SW1 to STM_WAKE1
Connections:
- net at U2.10 (PA4): no longer PMU_STATUS1.3 (DIN)
- net at U2.11 (PA5): now also PMU_STATUS1.3 (DIN)
Changed lines of the file:
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@@
+	)
+	(no_connect
+		(at 93.98 58.42)
 	)
 	(no_connect
 		(at 220.98 142.24)
 	)
-	(no_connect
-		(at 93.98 60.96)
-	)
 	(wire
 		(pts
@@
 	(wire
 		(pts
+			(xy 73.66 60.96) (xy 93.98 60.96)
+		)
+		(stroke
+			(width 0)
+			(type default)
+		)
+	)
+	(wire
+		(pts
+			(xy 73.66 60.96) (xy 73.66 93.98)
+		)
+		(stroke
+			(width 0)
+			(type default)
+		)
+	)
+	(wire
+		(pts
 			(xy 93.98 48.26) (xy 68.58 48.26)
 		)
@@
 	(wire
 		(pts
-			(xy 73.66 58.42) (xy 73.66 93.98)
-		)
-		(stroke
-			(width 0)
-			(type default)
-		)
-	)
-	(wire
-		(pts
 			(xy 88.9 63.5) (xy 93.98 63.5)
 		)
@@
 		(pts
 			(xy 160.02 68.58) (xy 160.02 73.66)
-		)
-		(stroke
-			(width 0)
-			(type default)
-		)
-	)
-	(wire
-		(pts
-			(xy 73.66 58.42) (xy 93.98 58.42)
 		)
 		(stroke
@@
 		(on_board yes)
 		(dnp no)
-		(property "Reference" "SW1"
+		(property "Reference" "STM_WAKE1"
 			(at 64.516 51.816 0)
 			(effects
@@
 			(project "bramble"
 				(path "/e35d7dcf-51bd-456f-89cf-e52d660079b4/df1d8afa-9717-44ff-901e-40cae4aada91"
-					(reference "SW1")
+					(reference "STM_WAKE1")
 					(unit 1)
 				)
@@
 		(dnp no)
 		(fields_autoplaced yes)
-		(property "Reference" "SW2"
+		(property "Reference" "STM_RESET1"
 			(at 189.23 55.88 0)
 			(effects
@@
 			(project "bramble"
 				(path "/e35d7dcf-51bd-456f-89cf-e52d660079b4/df1d8afa-9717-44ff-901e-40cae4aada91"
-					(reference "SW2")
+					(reference "STM_RESET1")
 					(unit 1)
 				)
@@
 			)
 		)
-		(property "Value" "MCP1700x-120xxMB"
+		(property "Value" "MCP1700T-3002E/MB"
 			(at 134.62 123.19 0)
 			(effects
@@
 			)
 		)
-		(property "Description" "250mA Low Quiscent Current LDO, 1.2V output, SOT-89"
+		(property "Description" "250mA Low Quiescent Current LDO, 3.0V output, SOT-89 (powers STM32L010 PMU)"
 			(at 134.62 127 0)
 			(effects
