File: schematics/hub-carrier-board/CM5.kicad_sch (KiCad schematic)
At the start: 4 parts, among them CN1 SM02B-SRSS-TB (LF)(SN), J101 ComputeModule5-CM5, J102 ComputeModule5-CM5, M303 Compute-Module-4_H1.5mm

Commit message: chore(schematics): update hub carrier board and add project file
Updates CM5/USB sub-sheets and the top-level hub-carrier-board
schematic. Also tracks hub-carrier-board.kicad_pro, which had only
been committed on the feat/hub-carrier-board branch.

Co-Authored-By: Claude Opus 4.7 (1M context) <noreply@anthropic.com>
Connections:
- net USB_PI.D_N is gone; now on net D-: J102.103 (USB2_N)
- net USB_PI.D_P is gone; now on net D+: J102.105 (USB2_P)
- net D+: no longer J102.134 (USB3-0-D_P)
- net D-: no longer J102.136 (USB3-0-D_N)
- new net USB.D+: J102.134 (USB3-0-D_P)
- new net USB.D-: J102.136 (USB3-0-D_N)
- no-connect marks 59 -> 58
Changed lines of the file:
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@@
 	)
 	(no_connect
-		(at 71.12 144.78)
-	)
-	(no_connect
 		(at 251.46 147.32)
 	)
@@
 	)
 	(bus_entry
-		(at 345.44 83.82)
-		(size -2.54 2.54)
-		(stroke
-			(width 0)
-			(type default)
-		)
-	)
-	(bus_entry
-		(at 342.9 83.82)
-		(size 2.54 -2.54)
-		(stroke
-			(width 0)
-			(type default)
-		)
-	)
-	(bus_entry
 		(at 242.57 83.82)
 		(size 2.54 2.54)
@@
 	)
 	(bus_entry
-		(at 342.9 86.36)
-		(size 2.54 -2.54)
-		(stroke
-			(width 0)
-			(type default)
-		)
-	)
-	(bus_entry
 		(at 351.79 106.68)
 		(size 2.54 -2.54)
@@
 	)
 	(bus_entry
-		(at 345.44 81.28)
-		(size -2.54 2.54)
-		(stroke
-			(width 0)
-			(type default)
-		)
-	)
-	(bus_entry
 		(at 237.49 175.26)
 		(size -2.54 2.54)
@@
 		)
 	)
-	(bus
-		(pts
-			(xy 345.44 81.28) (xy 345.44 83.82)
-		)
-		(stroke
-			(width 0)
-			(type default)
-		)
-	)
 	(wire
 		(pts
@@
 	(wire
 		(pts
-			(xy 71.12 144.78) (xy 86.36 144.78)
-		)
-		(stroke
-			(width 0)
-			(type solid)
-		)
-	)
-	(wire
-		(pts
 			(xy 328.93 190.5) (xy 347.98 190.5)
 		)
@@
 	(bus
 		(pts
-			(xy 345.44 72.39) (xy 345.44 81.28)
-		)
-		(stroke
-			(width 0)
-			(type default)
-		)
-	)
-	(bus
-		(pts
 			(xy 234.95 177.8) (xy 234.95 180.34)
 		)
@@
 	(wire
 		(pts
+			(xy 69.85 144.78) (xy 86.36 144.78)
+		)
+		(stroke
+			(width 0)
+			(type default)
+		)
+	)
+	(wire
+		(pts
 			(xy 147.32 147.32) (xy 161.29 147.32)
 		)
@@
 		)
 	)
-	(bus
-		(pts
-			(xy 345.44 72.39) (xy 344.17 72.39)
-		)
-		(stroke
-			(width 0)
-			(type default)
-		)
-	)
 	(wire
 		(pts
@@
 		)
 	)
-	(global_label "D-"
-		(shape input)
-		(at 238.76 124.46 180)
-		(fields_autoplaced yes)
-		(effects
-			(font
-				(size 1.27 1.27)
-			)
-			(justify right)
-		)
-		(property "Intersheetrefs" "${INTERSHEET_REFS}"
-			(at 232.9324 124.46 0)
-			(effects
-				(font
-					(size 1.27 1.27)
-				)
-				(justify right)
-				(hide yes)
-			)
-		)
-	)
 	(global_label "GPIO6"
 		(shape input)
@@
 	(global_label "D+"
 		(shape input)
-		(at 238.76 121.92 180)
+		(at 342.9 86.36 0)
 		(fields_autoplaced yes)
 		(effects
@@
 				(size 1.27 1.27)
 			)
-			(justify right)
+			(justify left)
 		)
 		(property "Intersheetrefs" "${INTERSHEET_REFS}"
-			(at 232.9324 121.92 0)
+			(at 348.7276 86.36 0)
 			(effects
 				(font
 					(size 1.27 1.27)
 				)
-				(justify right)
+				(justify left)
 				(hide yes)
 			)
@@
 		)
 	)
+	(global_label "D-"
+		(shape input)
+		(at 342.9 83.82 0)
+		(fields_autoplaced yes)
+		(effects
+			(font
+				(size 1.27 1.27)
+			)
+			(justify left)
+		)
+		(property "Intersheetrefs" "${INTERSHEET_REFS}"
+			(at 348.7276 83.82 0)
+			(effects
+				(font
+					(size 1.27 1.27)
+				)
+				(justify left)
+				(hide yes)
+			)
+		)
+	)
 	(global_label "GPIO5"
 		(shape input)
@@
 		)
 	)
-	(hierarchical_label "USB_PI{USB}"
-		(shape bidirectional)
-		(at 344.17 72.39 180)
-		(effects
-			(font
-				(size 1.27 1.27)
-			)
-			(justify right)
-		)
-	)
 	(hierarchical_label "ID_SC"
 		(shape output)
@@
 		(effects
 			(font
+				(size 1.27 1.27)
+			)
+			(justify right)
+		)
+	)
+	(hierarchical_label "GPIO4"
+		(shape input)
+		(at 69.85 144.78 180)
+		(effects
+			(font
