File: schematics/hub-carrier-board/USB.kicad_sch (KiCad schematic)
At the start: 10 parts, among them J5 USB_C_Receptacle_USB2.0_16P, U701 AP22653W6

Commit message: chore(schematics): update hub carrier board and add project file
Updates CM5/USB sub-sheets and the top-level hub-carrier-board
schematic. Also tracks hub-carrier-board.kicad_pro, which had only
been committed on the feat/hub-carrier-board branch.

Co-Authored-By: Claude Opus 4.7 (1M context) <noreply@anthropic.com>
Parts:
- removed C702: 100uF, Capacitor_Tantalum_SMD:CP_EIA-3528-21_Kemet-B, symbol Device:C_Polarized
- removed C703: 10u, Capacitor_SMD:C_0805_2012Metric, symbol Device:C
- removed R3: 15k, Resistor_SMD:R_0402_1005Metric, symbol Device:R_US
- removed U701: AP22653W6, Package_TO_SOT_SMD:SOT-23-6, symbol CM5IO:AP2553W6
- removed USB701: TYPEC-305-ACP16H458, EasyEDA:USB-C-SMD_TYPEC-305-ACP16H458, symbol EasyEDA:TYPEC-305-ACP16H458
- added C3: 100nF, Capacitor_SMD:C_0805_2012Metric_Pad1.18x1.45mm_HandSolder, symbol Device:C
- added C4: 100 uF, Capacitor_SMD:C_0805_2012Metric_Pad1.18x1.45mm_HandSolder, symbol Device:C
Connections:
- net VBUS is gone; now on net +5V: J5.A4 (VBUS), J5.A9 (VBUS), J5.B4 (VBUS), J5.B9 (VBUS)
- net +5V: now also C3.1, C4.1
- net D+: now also J5.B6 (D+)
- net D-: now also J5.B7 (D-)
- net GND: now also C3.2, C4.2
- no-connect marks 7 -> 2
Other:
- note removed: "Current Limit switch"
